File: BOARDS/mainProbe/mainProbe_ESP12_mill.sch (EAGLE design)
At the start: 18 parts

Commit message: placa com headers thanks to FS
Parts:
- renumbered U2 to DHT22
Changed lines of the file:
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@@
 <part name="D1" library="fab" deviceset="DIODE" device="SOD123"/>
 <part name="D2" library="fab" deviceset="DIODE" device="SOD123"/>
-<part name="U2" library="RHT03_DHT-22_AM2302" deviceset="RHT03_DHT-22_AM2302" device=""/>
+<part name="DHT22" library="RHT03_DHT-22_AM2302" deviceset="RHT03_DHT-22_AM2302" device=""/>
 <part name="TEMPSENSOR" library="headers(2mm)" deviceset="1X3" device=""/>
 <part name="R2" library="fab" deviceset="RES-US" device="1206" value="4.7K"/>
@@
 <instance part="D1" gate="G$1" x="68.58" y="83.82"/>
 <instance part="D2" gate="G$1" x="96.52" y="83.82"/>
-<instance part="U2" gate="G$1" x="157.48" y="83.82"/>
+<instance part="DHT22" gate="G$1" x="157.48" y="83.82"/>
 <instance part="TEMPSENSOR" gate="G$1" x="22.86" y="58.42"/>
 <instance part="R2" gate="G$1" x="30.48" y="48.26" rot="R90"/>
@@
 <net name="N$8" class="0">
 <segment>
-<pinref part="U2" gate="G$1" pin="DATA"/>
+<pinref part="DHT22" gate="G$1" pin="DATA"/>
 <wire x1="147.32" y1="86.36" x2="142.24" y2="86.36" width="0.1524" layer="91"/>
 <pinref part="R1" gate="G$1" pin="2"/>
@@
 </segment>
 <segment>
-<pinref part="U2" gate="G$1" pin="GND"/>
+<pinref part="DHT22" gate="G$1" pin="GND"/>
 <wire x1="147.32" y1="76.2" x2="121.92" y2="76.2" width="0.1524" layer="91"/>
 <label x="121.92" y="76.2" size="1.016" layer="95" rot="R180" xref="yes"/>
@@
 </segment>
 <segment>
-<pinref part="U2" gate="G$1" pin="VDD"/>
+<pinref part="DHT22" gate="G$1" pin="VDD"/>
 <wire x1="147.32" y1="91.44" x2="121.92" y2="91.44" width="0.1524" layer="91"/>
 <label x="121.92" y="91.44" size="1.016" layer="95" rot="R180" xref="yes"/>
