File: BOARDS/soilProbe/SoilProbe_ESP12.sch (EAGLE design)
At the start: 18 parts

Commit message: housekeeping over
Parts:
- removed JP1: (no value), pinhead:PINHD-1X4
- removed R1: 10K, fab:RES-US1206
Connections:
- removed net N$8: JP1.2, R1.2, U1.GPIO2
- net 3.3V: no longer JP1.1, JP1.3, R1.1
- net GND: no longer JP1.4
Changed lines of the file:
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@@
 <part name="U$1" library="fab" deviceset="FTDI-SMD-HEADER" device=""/>
 <part name="U$2" library="fab" deviceset="LED" device=""/>
-<part name="R1" library="fab" deviceset="RES-US" device="1206" value="10K"/>
 <part name="IC1" library="fab" deviceset="REGULATOR" device="SOT23"/>
 <part name="D1" library="fab" deviceset="DIODE" device="SOD123"/>
@@
 <part name="TEMPSENSOR" library="pinhead" library_urn="urn:adsk.eagle:library:325" deviceset="PINHD-1X3" device="" package3d_urn="urn:adsk.eagle:package:22458/2"/>
 <part name="SOLARIN" library="pinhead" library_urn="urn:adsk.eagle:library:325" deviceset="PINHD-1X2" device="/90" package3d_urn="urn:adsk.eagle:package:22437/2"/>
-<part name="JP1" library="pinhead" library_urn="urn:adsk.eagle:library:325" deviceset="PINHD-1X4" device="" package3d_urn="urn:adsk.eagle:package:22407/2"/>
 </parts>
 <sheets>
@@
 <instance part="U$1" gate="G$1" x="132.08" y="43.18"/>
 <instance part="U$2" gate="G$1" x="43.18" y="22.86" rot="R90"/>
-<instance part="R1" gate="G$1" x="137.16" y="86.36"/>
 <instance part="IC1" gate="G$1" x="25.4" y="86.36"/>
 <instance part="D1" gate="G$1" x="68.58" y="83.82"/>
@@
 <instance part="TEMPSENSOR" gate="A" x="20.32" y="58.42" rot="R180"/>
 <instance part="SOLARIN" gate="G$1" x="91.44" y="25.4" rot="R180"/>
-<instance part="JP1" gate="A" x="157.48" y="83.82"/>
 </instances>
 <busses>
@@
 <pinref part="U$1" gate="G$1" pin="TXD"/>
 <wire x1="132.08" y1="48.26" x2="124.46" y2="48.26" width="0.1524" layer="91"/>
-</segment>
-</net>
-<net name="N$8" class="0">
-<segment>
-<pinref part="R1" gate="G$1" pin="2"/>
-<wire x1="142.24" y1="86.36" x2="139.7" y2="86.36" width="0.1524" layer="91"/>
-<junction x="142.24" y="86.36"/>
-<wire x1="142.24" y1="86.36" x2="142.24" y2="81.28" width="0.1524" layer="91"/>
-<wire x1="142.24" y1="81.28" x2="111.76" y2="81.28" width="0.1524" layer="91"/>
-<wire x1="111.76" y1="81.28" x2="111.76" y2="45.72" width="0.1524" layer="91"/>
-<pinref part="U1" gate="G$1" pin="GPIO2"/>
-<wire x1="111.76" y1="45.72" x2="93.98" y2="45.72" width="0.1524" layer="91"/>
-<junction x="93.98" y="45.72"/>
-<pinref part="JP1" gate="A" pin="2"/>
-<wire x1="142.24" y1="86.36" x2="154.94" y2="86.36" width="0.1524" layer="91"/>
 </segment>
 </net>
@@
 </segment>
 <segment>
-<wire x1="154.94" y1="76.2" x2="121.92" y2="76.2" width="0.1524" layer="91"/>
-<label x="121.92" y="76.2" size="1.016" layer="95" rot="R180" xref="yes"/>
-<pinref part="JP1" gate="A" pin="4"/>
-<wire x1="154.94" y1="76.2" x2="154.94" y2="81.28" width="0.1524" layer="91"/>
-</segment>
-<segment>
 <pinref part="U$1" gate="G$1" pin="GND"/>
 <wire x1="132.08" y1="55.88" x2="124.46" y2="55.88" width="0.1524" layer="91"/>
@@
 </segment>
 <segment>
-<wire x1="154.94" y1="91.44" x2="121.92" y2="91.44" width="0.1524" layer="91"/>
-<label x="121.92" y="91.44" size="1.016" layer="95" rot="R180" xref="yes"/>
-<pinref part="R1" gate="G$1" pin="1"/>
-<wire x1="132.08" y1="86.36" x2="121.92" y2="86.36" width="0.1524" layer="91"/>
-<wire x1="121.92" y1="86.36" x2="121.92" y2="91.44" width="0.1524" layer="91"/>
-<junction x="121.92" y="91.44"/>
-<junction x="132.08" y="86.36"/>
-<pinref part="JP1" gate="A" pin="1"/>
-<wire x1="154.94" y1="91.44" x2="154.94" y2="88.9" width="0.1524" layer="91"/>
-<wire x1="154.94" y1="91.44" x2="165.1" y2="91.44" width="0.1524" layer="91"/>
-<wire x1="165.1" y1="91.44" x2="165.1" y2="83.82" width="0.1524" layer="91"/>
-<junction x="154.94" y="91.44"/>
-<pinref part="JP1" gate="A" pin="3"/>
-<wire x1="165.1" y1="83.82" x2="154.94" y2="83.82" width="0.1524" layer="91"/>
-</segment>
-<segment>
